File: Board/_saved_PlasmaTable.sch (KiCad schematic (older format))
At the start: 103 parts, among them CON1 BARREL_JACK, J1 USB, P1 CONN_5, P10 CONN_1, P11 CONN_1, P2 CONN_5, P3 CONN_5, P4 CONN_5, P5 CONN_5, P6 CONN_5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

Commit message: Just about finished routing
Parts:
- P1, P2, P3, P4, P5, P6, P7: footprint connect:SIL-5 -> PlasmaTable:PLUGABLE_HEADER
Changed lines of the file:
@@
 F 0 "P7" V 5000 7750 50  0000 C CNN
 F 1 "CONN_5" V 5100 7750 50  0000 C CNN
-F 2 "connect:SIL-5" H 5050 7750 60  0001 C CNN
+F 2 "PlasmaTable:PLUGABLE_HEADER" H 5050 7750 60  0001 C CNN
 F 3 "" H 5050 7750 60  0000 C CNN
 	1    5050 7750
@@
 F 0 "P6" V 4400 7750 50  0000 C CNN
 F 1 "CONN_5" V 4500 7750 50  0000 C CNN
-F 2 "connect:SIL-5" H 4450 7750 60  0001 C CNN
+F 2 "PlasmaTable:PLUGABLE_HEADER" H 4450 7750 60  0001 C CNN
 F 3 "" H 4450 7750 60  0000 C CNN
 	1    4450 7750
@@
 F 0 "P4" V 3200 7750 50  0000 C CNN
 F 1 "CONN_5" V 3300 7750 50  0000 C CNN
-F 2 "connect:SIL-5" H 3250 7750 60  0001 C CNN
+F 2 "PlasmaTable:PLUGABLE_HEADER" H 3250 7750 60  0001 C CNN
 F 3 "" H 3250 7750 60  0000 C CNN
 	1    3250 7750
@@
 F 0 "P3" V 2550 7750 50  0000 C CNN
 F 1 "CONN_5" V 2650 7750 50  0000 C CNN
-F 2 "connect:SIL-5" H 2600 7750 60  0001 C CNN
+F 2 "PlasmaTable:PLUGABLE_HEADER" H 2600 7750 60  0001 C CNN
 F 3 "" H 2600 7750 60  0000 C CNN
 	1    2600 7750
@@
 F 0 "P1" V 1250 7750 50  0000 C CNN
 F 1 "CONN_5" V 1350 7750 50  0000 C CNN
-F 2 "connect:SIL-5" H 1300 7750 60  0001 C CNN
+F 2 "PlasmaTable:PLUGABLE_HEADER" H 1300 7750 60  0001 C CNN
 F 3 "" H 1300 7750 60  0000 C CNN
 	1    1300 7750
@@
 F 0 "P5" V 3800 7750 50  0000 C CNN
 F 1 "CONN_5" V 3900 7750 50  0000 C CNN
-F 2 "connect:SIL-5" H 3850 7750 60  0001 C CNN
+F 2 "PlasmaTable:PLUGABLE_HEADER" H 3850 7750 60  0001 C CNN
 F 3 "" H 3850 7750 60  0000 C CNN
 	1    3850 7750
@@
 F 0 "P2" V 1900 7750 50  0000 C CNN
 F 1 "CONN_5" V 2000 7750 50  0000 C CNN
-F 2 "connect:SIL-5" H 1950 7750 60  0001 C CNN
+F 2 "PlasmaTable:PLUGABLE_HEADER" H 1950 7750 60  0001 C CNN
 F 3 "" H 1950 7750 60  0000 C CNN
 	1    1950 7750
