File: Board/PlasmaTable.kicad_pcb (KiCad board)
At the start: 2 copper layers, 152.4 x 104.1 mm, 103 parts, among them CON1 BARREL_JACK, J1 USB, P1 CONN_5, P10 CONN_1, P11 CONN_1, P2 CONN_5, P3 CONN_5, P4 CONN_5, P5 CONN_5, P6 CONN_5, P7 CONN_5, P8 CONN_1, P9 CONN_1, Q1 DARL_N, Q2 DARL_N, Q3 DARL_N, Q4 DARL_N, Q5 DARL_N, U1 PHOTON, U2 7805, U3 7805, U4 7805, U5 7805

Commit message: Finished Roughting
Parts:
- added C39: C, smd_capacitors:c_0603, F.Cu at (88.1, 80.4)
Routing:
- net GND: track 724.2 -> 1116.2 mm, vias 19 -> 34
- net +3.3V: track 0.00 -> 239.0 mm
- net /SWITCH1: track 27.0 -> 209.9 mm, vias 0 -> 4
- net /SWITCH3: track 16.8 -> 175.9 mm, vias 0 -> 3
- net /SWITCH2: track 21.7 -> 180.6 mm, vias 0 -> 3
- net /DRV_ENABLE: track 0.00 -> 158.6 mm, vias 0 -> 2
- net /SWITCH4: track 14.7 -> 171.0 mm, vias 0 -> 3
- net /SWITCH5: track 13.0 -> 166.6 mm, vias 1 -> 4
- net /SWITCH6: track 0.00 -> 151.5 mm, vias 0 -> 5
- net +24V: track 437.4 -> 521.5 mm, vias 7 -> 14
- net +5V: track 206.3 -> 279.4 mm
- net Net-(DRV3-Pad5): track 0.00 -> 46.7 mm, vias 0 -> 2
- net Net-(DRV2-Pad5): track 0.00 -> 30.6 mm, vias 0 -> 1
- net Net-(DRV1-Pad5): track 0.00 -> 28.2 mm, vias 0 -> 1
- net Net-(DRV2-Pad23): track 58.3 -> 49.1 mm
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